Commit message: Modify forward multibeam sonar for nekton

File: uuv_sensor_plugins/uuv_sensor_ros_plugins/urdf/sonar_snippets.xacro (robot description, xacro)
@@ -76,10 +76,10 @@
     </xacro:multibeam_sonar>
   </xacro:macro>
-  <xacro:macro name="forward_multibeam_p900" params="namespace parent_link *origin">
+  <xacro:macro name="forward_multibeam_p900" params="namespace parent_link topic *origin">
     <xacro:multibeam_sonar
       namespace="${namespace}"
       suffix=""
       parent_link="${parent_link}"
-      topic="sonar"
+      topic="${topic}"
       mass="0.02"
       update_rate="15"
@@ -113,5 +113,5 @@
       <xacro:no_collision/>
     </link>
-  <joint name="${namespace}_sonar${suffix}_joint" type="revolute">
+  <joint name="${namespace}_sonar${suffix}_joint" type="fixed">
     <xacro:insert_block name="origin" />
     <parent link="${parent_link}" />
@@ -121,5 +121,5 @@
   </joint>
   <gazebo reference="${namespace}/sonar${suffix}_link">
-    <sensor type="gpu_ray" name="sonar${suffix}">
+    <sensor type="ray" name="sonar${suffix}">
       <pose>0 0 0 0 0 0</pose>
       <visualize>false</visualize>
@@ -145,6 +145,8 @@
         </noise>
       </ray>
-      <plugin name="sonar${suffix}_controller" filename="libgazebo_ros_gpu_laser.so">
-        <topicName>${topic}</topicName>
+      <plugin name="sonar${suffix}_controller" filename="libgazebo_ros_ray_sensor.so">
+        <ros>
+	  <remapping>~\out:${topic}</remapping>
+	</ros>
         <frameName>sonar${suffix}_link</frameName>
       </plugin>

Commit message: Fix sonar offset issue

File: uuv_sensor_plugins/uuv_sensor_ros_plugins/urdf/sonar_snippets.xacro (robot description, xacro)
@@ -113,5 +113,5 @@
       <xacro:no_collision/>
     </link>
-  <joint name="${namespace}_sonar${suffix}_joint" type="fixed">
+  <joint name="${namespace}_sonar${suffix}_joint" type="revolute">
     <xacro:insert_block name="origin" />
     <parent link="${parent_link}" />
