Commit message: Add topic name to default camera

File: uuv_sensor_plugins/uuv_sensor_ros_plugins/urdf/camera_snippets.xacro (robot description, xacro)
@@ -27,10 +27,10 @@
     </collision>
   </xacro:macro>
-  <xacro:macro name="default_camera" params="namespace parent_link suffix *origin">
+  <xacro:macro name="default_camera" params="namespace parent_link suffix topic *origin">
     <xacro:regular_camera_plugin_macro
       namespace="${namespace}"
       suffix="${suffix}"
       parent_link="${parent_link}"
-      topic="camera"
+      topic="${topic}"
       mass="0.1"
       update_rate="30"
